File: Eagle/Version2/Jeep_ECU.brd (EAGLE design)
At the start: 34.8 x 66.5 mm, 32 parts, among them Q1 NPN-TRANSISTORMMBT3904-SOT23

Commit message: Updated BOM
Parts:
- renumbered U$2 to UPS1
Changed lines of the file:
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@@
 </autorouter>
 <elements>
-<element name="U$1" library="Eberle" package="MOLEX_15PIN_BOARD" value="MOLEX_15_BOARD" x="15.748" y="49.276"/>
+<element name="U$1" library="Eberle" package="MOLEX_15PIN_BOARD" value="MOLEX_15_BOARD" x="15.748" y="49.276">
+<attribute name="MFG" value="Molex" x="15.748" y="49.276" size="1.778" layer="27" display="off"/>
+<attribute name="PN" value="03-09-2151 / 02-09-2134 " x="15.748" y="49.276" size="1.778" layer="27" display="off"/>
+</element>
 <element name="CPS6" library="Eberle" package="0603-CAP" value="0.1u" x="19.558" y="31.496" smashed="yes" rot="R180">
 <attribute name="MFG" value="Vishay" x="36.068" y="-15.494" size="1.778" layer="27" rot="R180" display="off"/>
@@
 <attribute name="VDC" value="16" x="27.94" y="34.544" size="1.778" layer="27" rot="R180" display="off"/>
 </element>
-<element name="U$2" library="Eberle" package="17395XX78" value="17395XX78173950578" x="10.414" y="25.146"/>
+<element name="UPS1" library="Eberle" package="17395XX78" value="17395XX78173950578" x="10.414" y="25.146">
+<attribute name="MFG" value="Wurth" x="10.414" y="25.146" size="1.778" layer="27" display="off"/>
+<attribute name="PN" value="173950578" x="10.414" y="25.146" size="1.778" layer="27" display="off"/>
+</element>
 <element name="C3" library="Eberle" package="8X10MM-ELECTROLYTIC" value="330u" x="9.398" y="17.272" rot="R90">
 <attribute name="MFG" value="Nichicon" x="9.398" y="17.272" size="1.778" layer="27" rot="R90" display="off"/>
 <attribute name="PN" value="UCL1E331MNL1GS" x="9.398" y="17.272" size="1.778" layer="27" rot="R90" display="off"/>
+<attribute name="VDC" value="25" x="9.398" y="17.272" size="1.778" layer="27" rot="R90" display="off"/>
 </element>
 <element name="TP_12V" library="Eberle" package="TEST_POINT" value="TEST_POINT" x="1.778" y="27.178" smashed="yes">
@@
 <via x="32.258" y="41.148" extent="1-16" drill="0.35"/>
 <wire x1="32.258" y1="41.148" x2="24.892" y2="41.148" width="0.508" layer="16"/>
-<contactref element="U$2" pad="GND"/>
+<contactref element="UPS1" pad="GND"/>
 <contactref element="C3" pad="-"/>
 <wire x1="19.05" y1="35.56" x2="16.256" y2="32.766" width="0.8128" layer="16"/>
@@
 <contactref element="DPS3" pad="C"/>
 <contactref element="DPS4" pad="C"/>
-<contactref element="U$2" pad="VIN"/>
+<contactref element="UPS1" pad="VIN"/>
 <contactref element="C3" pad="+"/>
 <contactref element="TP_12V" pad="P$1"/>
@@
 <wire x1="24.892" y1="31.496" x2="24.892" y2="51.982" width="0.508" layer="1"/>
 <wire x1="25.9842" y1="29.21" x2="24.892" y2="29.21" width="0.508" layer="1"/>
-<contactref element="U$2" pad="VOUT"/>
+<contactref element="UPS1" pad="VOUT"/>
 <wire x1="12.954" y1="25.146" x2="12.954" y2="27.178" width="0.762" layer="16"/>
 <wire x1="12.954" y1="27.178" x2="14.224" y2="28.448" width="0.762" layer="16"/>
