File: Eagle/Version2/Jeep_ECU.sch (EAGLE design)
At the start: 32 parts, among them Q1 NPN-TRANSISTORMMBT3904-SOT23

Commit message: Updated BOM
Parts:
- C3: VDC (none) -> 25
- U$1: MFG (none) -> Molex; PN (none) -> 03-09-2151 / 02-09-2134
- UPS1: MFG (none) -> Wurth; PN (none) -> 173950578
- renumbered U$2 to UPS1
Changed lines of the file:
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@@
 </classes>
 <parts>
-<part name="U$1" library="Eberle" deviceset="MOLEX_15_BOARD" device=""/>
+<part name="U$1" library="Eberle" deviceset="MOLEX_15_BOARD" device="">
+<attribute name="MFG" value="Molex"/>
+<attribute name="PN" value="03-09-2151 / 02-09-2134 "/>
+</part>
 <part name="CPS6" library="Eberle" deviceset="CAP" device="0606-CAP" value="0.1u">
 <attribute name="MFG" value="Vishay"/>
@@
 <attribute name="VDC" value="16"/>
 </part>
-<part name="U$2" library="Eberle" deviceset="17395XX78" device="173950578"/>
+<part name="UPS1" library="Eberle" deviceset="17395XX78" device="173950578">
+<attribute name="MFG" value="Wurth"/>
+<attribute name="PN" value="173950578"/>
+</part>
 <part name="C3" library="Eberle" deviceset="CAP_POLTH1_JE" device="8X10MM-SMD" value="330u">
 <attribute name="MFG" value="Nichicon"/>
 <attribute name="PN" value="UCL1E331MNL1GS"/>
+<attribute name="VDC" value="25"/>
 </part>
 <part name="TP_12V" library="Eberle" deviceset="TEST_POINT" device=""/>
@@
 <sheet>
 <plain>
-<text x="-116.84" y="195.58" size="1.778" layer="91">V2 Changes
+<text x="12.7" y="147.32" size="1.778" layer="91">V2 Changes
 - 470u Input CAP
 - TP on transistor Output
@@
 </plain>
 <instances>
-<instance part="U$1" gate="G$1" x="2.54" y="25.4"/>
+<instance part="U$1" gate="G$1" x="2.54" y="25.4">
+<attribute name="MFG" x="2.54" y="25.4" size="1.778" layer="96" display="off"/>
+<attribute name="PN" x="2.54" y="25.4" size="1.778" layer="96" display="off"/>
+</instance>
 <instance part="CPS6" gate="G$1" x="195.58" y="91.44" smashed="yes">
 <attribute name="NAME" x="198.12" y="90.17" size="1.778" layer="95"/>
@@
 <attribute name="VDC" x="276.86" y="127" size="1.778" layer="96" display="off"/>
 </instance>
-<instance part="U$2" gate="G$1" x="144.78" y="99.06"/>
+<instance part="UPS1" gate="G$1" x="144.78" y="99.06">
+<attribute name="MFG" x="144.78" y="99.06" size="1.778" layer="96" display="off"/>
+<attribute name="PN" x="144.78" y="99.06" size="1.778" layer="96" display="off"/>
+</instance>
 <instance part="C3" gate="G$1" x="106.68" y="93.98">
 <attribute name="MFG" x="106.68" y="93.98" size="1.778" layer="96" display="off"/>
 <attribute name="PN" x="106.68" y="93.98" size="1.778" layer="96" display="off"/>
+<attribute name="VDC" x="106.68" y="93.98" size="1.778" layer="96" display="off"/>
 </instance>
 <instance part="TP_12V" gate="G$1" x="83.82" y="116.84" rot="R90">
@@
 <wire x1="195.58" y1="78.74" x2="218.44" y2="78.74" width="0.1524" layer="91"/>
 <junction x="195.58" y="78.74"/>
-<pinref part="U$2" gate="G$1" pin="GND/ADJ"/>
+<pinref part="UPS1" gate="G$1" pin="GND/ADJ"/>
 <wire x1="144.78" y1="91.44" x2="144.78" y2="78.74" width="0.1524" layer="91"/>
 <junction x="144.78" y="78.74"/>
@@
 <pinref part="DPS3" gate="G$1" pin="C"/>
 <pinref part="DPS4" gate="G$1" pin="C"/>
-<pinref part="U$2" gate="G$1" pin="VI"/>
+<pinref part="UPS1" gate="G$1" pin="VI"/>
 <pinref part="C3" gate="G$1" pin="+"/>
 <wire x1="134.62" y1="99.06" x2="106.68" y2="99.06" width="0.1524" layer="91"/>
@@
 <wire x1="180.34" y1="106.68" x2="180.34" y2="99.06" width="0.1524" layer="91"/>
 <junction x="180.34" y="99.06"/>
-<pinref part="U$2" gate="G$1" pin="VO"/>
-</segment>
-<segment>
+<pinref part="UPS1" gate="G$1" pin="VO"/>
+</segment>
+<segment>
